File: pcb/centronics.kicad_sch (KiCad schematic)
At the start: 5 parts, among them J1 Conn_02x15_Row_Letter_Last, U1 74LS138, U2 74LS138, U3 74LS374, U4 74LS367

Commit message: Expanding schematic
Parts:
- added J2: top connector, symbol Connector:Conn_01x15_Pin
- added R1, R2, R3, R4, R5: 2k2, symbol Device:R
- added U5: 74LS165, symbol 74xx:74LS165
- J1: value Conn_02x15_Row_Letter_Last -> P2000T SLOT2
Connections:
- net 2.5MHz: now also U5.2 (CP)
- net CP: now also U5.1 (~{PL})
- net D0: now also U4.9 (O4a)
- net D1: now also U3.14 (D5), U4.11 (O5b)
- net D2: now also U3.17 (D6), U4.13 (O6b)
- net D3: now also U3.8 (D3), U4.7 (O3a)
- net D4: now also U3.7 (D2), U4.5 (O2a)
- net D5: now also U3.4 (D1), U4.2 (I1), U4.3 (O1a)
- net D6: now also U3.18 (D7)
- net D7: now also U3.3 (D0)
- net GND: now also U3.1 (OE), U5.4 (D5), U5.5 (D6), U5.6 (D7), U5.8 (GND)
- net VCC: now also R1.2, R2.2, R3.2, R4.2, R5.2, U5.11 (D0), U5.12 (D1), U5.13 (D2), U5.14 (D3), U5.16 (VCC)
- net 10: now reaches U4.10 (I4)
- net 10: now also J2.10 (Pin_10), R2.1
- net 11: now reaches U4.12 (I5)
- net 11: now also J2.11 (Pin_11), R3.1
- net 12: now reaches U4.14 (I6)
- net 12: now also J2.12 (Pin_12), R4.1
- net 32: now reaches U4.4 (I2)
- net 32: now also J2.15 (Pin_15), R5.1
- net 13: now reaches U4.6 (I3)
- net 13: now also J2.13 (Pin_13), R1.1
- net 2: now reaches U3.12 (O4)
- net 2: now also J2.2 (Pin_2)
- net 3: now reaches U3.15 (O5)
- net 3: now also J2.3 (Pin_3)
- net 4: now reaches U3.16 (O6)
- net 4: now also J2.4 (Pin_4)
- net 8: now reaches U3.19 (O7)
- net 8: now also J2.8 (Pin_8)
- net 9: now reaches U3.2 (O0)
- net 9: now also J2.9 (Pin_9)
- net 7: now reaches U3.5 (O1)
- net 7: now also J2.7 (Pin_7)
- net 6: now reaches U3.6 (O2)
- net 6: now also J2.6 (Pin_6)
- net 5: now reaches U3.9 (O3)
- net 5: now also J2.5 (Pin_5)
- new net 1: J2.1 (Pin_1), U5.7 (~{Q7})
- new net 14: J2.14 (Pin_14)
- no-connect marks 20 -> 24
Other:
- note added: "Should be connected to GND?"

Commit message: Making corrections
Connections:
- net GND: now also U5.10 (DS)
- net VCC: now also U5.3 (D4)
- no-connect marks 24 -> 22
Other:
- note added: "76543210 ~{WR} ~{IOREQ} X100011X X 0"
- note added: "76543210 ~{WR} ~{IOREQ} ~{M1} 01000111 0 0 1 0x47 WRITE"
- note added: "76543210 ~{WR} ~{IOREQ} ~{M1} 01000111 1 0 1 0x47 READ"
- note removed: "76543210 ~{WR} ~{IOREQ} 1100011X X 0"
- note removed: "76543210 ~{WR} ~{IOREQ} ~{M1} 11000111 0 0 1 0xC7 WRITE"
- note removed: "76543210 ~{WR} ~{IOREQ} ~{M1} 11000111 1 0 1 0xC7 READ"
Changed lines of the file:
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@@
 	)
 	(junction
-		(at 190.5 92.71)
+		(at 190.5 96.52)
 		(diameter 0)
 		(color 0 0 0 0)
@@
 	)
 	(no_connect
-		(at 193.04 86.36)
-	)
-	(no_connect
 		(at 66.04 40.64)
 	)
 	(no_connect
-		(at 193.04 99.06)
-	)
-	(no_connect
 		(at 83.82 160.02)
 	)
@@
 	(wire
 		(pts
-			(xy 190.5 92.71) (xy 190.5 91.44)
+			(xy 190.5 91.44) (xy 190.5 93.98)
 		)
 		(stroke
@@
 	(wire
 		(pts
+			(xy 190.5 99.06) (xy 190.5 96.52)
+		)
+		(stroke
+			(width 0)
+			(type default)
+		)
+	)
+	(wire
+		(pts
 			(xy 193.04 101.6) (xy 190.5 101.6)
 		)
@@
 	(wire
 		(pts
-			(xy 190.5 104.14) (xy 193.04 104.14)
+			(xy 193.04 99.06) (xy 190.5 99.06)
 		)
 		(stroke
@@
 	(wire
 		(pts
-			(xy 105.41 110.49) (xy 107.95 110.49)
+			(xy 190.5 104.14) (xy 193.04 104.14)
 		)
 		(stroke
@@
 	(wire
 		(pts
-			(xy 161.29 92.71) (xy 158.75 92.71)
+			(xy 105.41 110.49) (xy 107.95 110.49)
 		)
 		(stroke
@@
 	(wire
 		(pts
-			(xy 190.5 106.68) (xy 193.04 106.68)
+			(xy 161.29 92.71) (xy 158.75 92.71)
 		)
 		(stroke
@@
 	(wire
 		(pts
-			(xy 107.95 110.49) (xy 107.95 111.76)
+			(xy 190.5 106.68) (xy 193.04 106.68)
 		)
 		(stroke
@@
 	(wire
 		(pts
-			(xy 161.29 102.87) (xy 165.1 102.87)
+			(xy 107.95 110.49) (xy 107.95 111.76)
 		)
 		(stroke
@@
 	(wire
 		(pts
-			(xy 190.5 96.52) (xy 193.04 96.52)
+			(xy 161.29 102.87) (xy 165.1 102.87)
 		)
 		(stroke
@@
 	(wire
 		(pts
-			(xy 190.5 92.71) (xy 190.5 93.98)
+			(xy 190.5 96.52) (xy 193.04 96.52)
 		)
 		(stroke
@@
 		)
 	)
-	(text "76543210 ~{WR} ~{IOREQ} ~{M1}\n11000111  1  0      1\n0xC7\nREAD"
+	(text "76543210 ~{WR} ~{IOREQ} ~{M1}\n01000111  1  0      1\n0x47\nREAD"
 		(exclude_from_sim no)
 		(at 72.39 56.642 0)
@@
 		)
 	)
-	(text "76543210 ~{WR} ~{IOREQ}\n1100011X  X  0"
+	(text "76543210 ~{WR} ~{IOREQ}\nX100011X  X  0"
 		(exclude_from_sim no)
 		(at 137.922 39.37 0)
@@
 		)
 	)
-	(text "76543210 ~{WR} ~{IOREQ} ~{M1}\n11000111  0  0      1\n0xC7\nWRITE"
+	(text "76543210 ~{WR} ~{IOREQ} ~{M1}\n01000111  0  0      1\n0x47\nWRITE"
 		(exclude_from_sim no)
 		(at 72.39 43.434 0)
@@
 	(symbol
 		(lib_id "power:VCC")
-		(at 190.5 92.71 90)
+		(at 190.5 93.98 90)
 		(unit 1)
 		(exclude_from_sim no)
@@
 		(fields_autoplaced yes)
 		(property "Reference" "#PWR017"
-			(at 194.31 92.71 0)
+			(at 194.31 93.98 0)
 			(effects
 				(font
@@
 		)
 		(property "Value" "VCC"
-			(at 186.69 92.7099 90)
+			(at 186.69 93.9799 90)
 			(effects
 				(font
@@
 		)
 		(property "Footprint" ""
-			(at 190.5 92.71 0)
+			(at 190.5 93.98 0)
 			(effects
 				(font
@@
 		)
 		(property "Datasheet" ""
-			(at 190.5 92.71 0)
+			(at 190.5 93.98 0)
 			(effects
 				(font
@@
 		)
 		(property "Description" "Power symbol creates a global label with name \"VCC\""
-			(at 190.5 92.71 0)
+			(at 190.5 93.98 0)
 			(effects
 				(font
@@
 					(unit 1)
 				)
+			)
+		)
+	)
+	(symbol
+		(lib_id "power:GND")
+		(at 193.04 86.36 270)
+		(unit 1)
+		(exclude_from_sim no)
+		(in_bom yes)
+		(on_board yes)
+		(dnp no)
+		(fields_autoplaced yes)
+		(property "Reference" "#PWR018"
+			(at 186.69 86.36 0)
+			(effects
+				(font
+					(size 1.27 1.27)
+				)
+				(hide yes)
+			)
+		)
+		(property "Value" "GND"
+			(at 189.23 86.3599 90)
+			(effects
+				(font
+					(size 1.27 1.27)
+				)
+				(justify right)
+			)
+		)
+		(property "Footprint" ""
+			(at 193.04 86.36 0)
+			(effects
+				(font
+					(size 1.27 1.27)
+				)
+				(hide yes)
+			)
+		)
+		(property "Datasheet" ""
+			(at 193.04 86.36 0)
+			(effects
+				(font
+					(size 1.27 1.27)
+				)
+				(hide yes)
+			)
+		)
+		(property "Description" "Power symbol creates a global label with name \"GND\" , ground"
+			(at 193.04 86.36 0)
+			(effects
+				(font
+					(size 1.27 1.27)
+				)
+				(hide yes)
+			)
+		)
+		(pin "1"
+		)
+		(instances
+			(project "centronics"
+				(path "/fed2f63f-e834-4b73-8e0d-0fc3a743b9a8"
+					(reference "#PWR018")
+					(unit 1)
+				)
